File: pcb/reflow-example/reflow-example.kicad_sch (KiCad schematic)
At the start: 50 parts, among them IC1 CD4511BNSR, IC2 CD4511BNSR, U1 NE555D, U4 74LS393

Commit message: update:
Parts:
- removed U4: 74LS393, Package_DIP:DIP-14_W7.62mm_SMDSocket_SmallPads, symbol 74xx:74LS393
- removed V1: 5, Connector_PinHeader_2.54mm:PinHeader_1x02_P2.54mm_Horizontal, symbol Simulation_SPICE:VDC
- added J1: USB_C_Receptacle_PowerOnly_6P, Connector_USB:USB_C_Receptacle_GCT_USB4135-GF-A_6P_TopMnt_Horizontal, symbol Connector:USB_C_Receptacle_PowerOnly_6P
- added R17, R18: 5k1, Capacitor_SMD:C_1206_3216Metric, symbol Device:R_US
- added U2: 4518, Package_DIP:DIP-16_W8.89mm_SMDSocket_LongPads, symbol 4xxx:4518
Connections:
- net +5V: now also J1.A9 (VBUS), J1.B9 (VBUS), U2.10 (Enable), U2.16 (VDD), U2.2 (Enable)
- net GND: now also J1.A12 (GND), J1.B12 (GND), J1.S1 (SHIELD), R17.2, R18.2, U2.15 (Reset), U2.7 (Reset), U2.8 (VSS)
- net at IC2.1 (B_1): now also U2.12 (Q2)
- net at IC2.7 (A_1): now also U2.11 (Q1)
- net at U1.3 (Q): now also U2.1 (CK), U2.9 (CK)
- net at IC2.6 (D_1): now also U2.14 (Q4)
- net at IC2.2 (C_1): now also U2.13 (Q3)
- net at IC1.1 (B_1): now also U2.4 (Q2)
- net at IC1.2 (C_1): now also U2.5 (Q3)
- net at IC1.6 (D_1): now also U2.6 (Q4)
- net at IC1.7 (A_1): now also U2.3 (Q1)
- new net: J1.A5 (CC1), R17.1
- new net: J1.B5 (CC2), R18.1
